File: badge.sch (KiCad schematic (older format))
At the start: 2 parts, among them J1 Conn_01x40_Female, U1 ESP32-DEVKITC-32D

Commit message: Add btn, jumpers
Parts:
- removed J1: Conn_01x40_Female, Connector_FFC-FPC:Hirose_FH12-40S-0.5SH_1x40-1MP_P0.50mm_Horizontal, symbol Connector:Conn_01x40_Female
- added C1, C2, C3, C4, C5, C6, C7: 0.1uF, Capacitor_SMD:C_0603_1608Metric, symbol Device:C_Small
- added J1: DevKitC_L, Connector_PinHeader_2.54mm:PinHeader_1x20_P2.54mm_Vertical_SMD_Pin1Right, symbol Connector:Conn_01x20_Female
- added J2: DevKitC_R, Connector_PinHeader_2.54mm:PinHeader_1x20_P2.54mm_Vertical_SMD_Pin1Right, symbol Connector:Conn_01x20_Female
- added J3: HT024SQV010NH, Connector_FFC-FPC:Hirose_FH12-40S-0.5SH_1x40-1MP_P0.50mm_Horizontal, symbol New_Library:HT024SQV010NH
- added J4: EXT1_1, Connector_PinHeader_2.54mm:PinHeader_1x04_P2.54mm_Vertical, symbol Connector:Conn_01x04_Female
- added J5: EXT1_2, Connector_PinHeader_2.54mm:PinHeader_1x04_P2.54mm_Vertical, symbol Connector:Conn_01x04_Female
- added J6: EXT1_3, Connector_PinHeader_2.54mm:PinHeader_1x04_P2.54mm_Vertical, symbol Connector:Conn_01x04_Female
- added J7: EXT2_1, Connector_PinHeader_2.54mm:PinHeader_1x06_P2.54mm_Vertical, symbol Connector:Conn_01x06_Female
- added J8: EXT2_2, Connector_PinHeader_2.54mm:PinHeader_1x06_P2.54mm_Vertical, symbol Connector:Conn_01x06_Female
- added J9: EXT2_3, Connector_PinHeader_2.54mm:PinHeader_1x06_P2.54mm_Vertical, symbol Connector:Conn_01x06_Female
- added R1, R2, R3: 0603/12R, Resistor_SMD:R_0603_1608Metric, symbol Device:R_Small
- added SW1: UP, Button_Switch_SMD:SW_SPST_TL3342, symbol Switch:SW_Push
- added SW2: LEFT, Button_Switch_SMD:SW_SPST_TL3342, symbol Switch:SW_Push
- added SW3: A, Button_Switch_SMD:SW_SPST_TL3342, symbol Switch:SW_Push
- added SW4: DOWN, Button_Switch_SMD:SW_SPST_TL3342, symbol Switch:SW_Push
- added SW5: RIGHT, Button_Switch_SMD:SW_SPST_TL3342, symbol Switch:SW_Push
- added SW6: B, Button_Switch_SMD:SW_SPST_TL3342, symbol Switch:SW_Push
Connections:
- net labels added: +3.3V, +5V, GND, GPIO12, GPIO13, GPIO14, GPIO15, GPIO25, GPIO26, GPIO27, GPIO34, GPIO35, GPIO36, GPIO39, GPIO4, LCD_DC, LCD_RST, VSPI_CS, VSPI_MISO, VSPI_MOSI, VSPI_SCK
- wire segments 0 -> 92
- no-connect marks 0 -> 32
Other:
- moved on the sheet: U1

Commit message: Change to manual PCB
Parts:
- added C8: 0.1uF, Capacitor_SMD:C_0603_1608Metric, symbol Device:C_Small
- added H1, H2: MountingHole, MountingHole:MountingHole_5mm, symbol Mechanical:MountingHole
- added J10: HT024SQV003NH, custom_footprint:COMMON_MOUNT_FFC-1x18-1MP_P0.80mm, symbol New_Library:HT024SQV003NH
- added R4: 0603/4.7, Resistor_SMD:R_0603_1608Metric, symbol Device:R_Small
- J1, J2: footprint Connector_PinHeader_2.54mm:PinHeader_1x20_P2.54mm_Vertical_SMD_Pin1Right -> Connector_PinHeader_2.54mm:PinHeader_1x20_P2.54mm_Vertical
- R1, R2, R3: value 0603/12R -> 0603/10R
Connections:
- wire segments 92 -> 106
- no-connect marks 32 -> 36
Other:
- moved on the sheet: C2, C3, C4, C5, C6, C7, SW1, SW2, SW3, SW4, SW5, SW6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

Commit message: Square layout
Parts:
- added N1: Housing, custom_footprint:2.4INCH_TFT_LCD_18P_0.80mm_FOLD, symbol Mechanical:Housing
- J1, J2: footprint Connector_PinHeader_2.54mm:PinHeader_1x20_P2.54mm_Vertical -> Connector_PinSocket_2.54mm:PinSocket_1x19_P2.54mm_Vertical; symbol Connector:Conn_01x20_Female -> Connector:Conn_01x19_Female
- J4, J5, J6: footprint Connector_PinHeader_2.54mm:PinHeader_1x04_P2.54mm_Vertical -> Connector_PinSocket_2.54mm:PinSocket_1x04_P2.54mm_Vertical
- J7, J8, J9: footprint Connector_PinHeader_2.54mm:PinHeader_1x06_P2.54mm_Vertical -> Connector_PinSocket_2.54mm:PinSocket_1x06_P2.54mm_Vertical
- U1: footprint ESP32-DEVKITC-32D:MODULE_ESP32-DEVKITC-32D -> custom_footprint:MODULE_ESP32-DEVKITC-32D-SILKONLY
Changed lines of the file:
@@
 F 0 "U1" H 2300 3167 50  0000 C CNN
 F 1 "ESP32-DEVKITC-32D" H 2300 3076 50  0000 C CNN
-F 2 "ESP32-DEVKITC-32D:MODULE_ESP32-DEVKITC-32D" H 2300 2000 50  0001 L BNN
+F 2 "custom_footprint:MODULE_ESP32-DEVKITC-32D-SILKONLY" H 2300 2000 50  0001 L BNN
 F 3 "None" H 2300 2000 50  0001 L BNN
 F 4 "Espressif Systems" H 2300 2000 50  0001 L BNN "Field4"
@@
 LCD_DC
 $Comp
-L Connector:Conn_01x20_Female J1
+L Connector:Conn_01x19_Female J1
 U 1 1 5BD639DE
 P 1400 2000
 F 0 "J1" H 1300 3100 50  0000 L CNN
 F 1 "DevKitC_L" H 1100 3000 50  0000 L CNN
-F 2 "Connector_PinHeader_2.54mm:PinHeader_1x20_P2.54mm_Vertical" H 1400 2000 50  0001 C CNN
+F 2 "Connector_PinSocket_2.54mm:PinSocket_1x19_P2.54mm_Vertical" H 1400 2000 50  0001 C CNN
 F 3 "~" H 1400 2000 50  0001 C CNN
 	1    1400 2000
@@
 $EndComp
 $Comp
-L Connector:Conn_01x20_Female J2
+L Connector:Conn_01x19_Female J2
 U 1 1 5BD63A56
 P 3200 2000
 F 0 "J2" H 3094 3085 50  0000 C CNN
 F 1 "DevKitC_R" H 3094 2994 50  0000 C CNN
-F 2 "Connector_PinHeader_2.54mm:PinHeader_1x20_P2.54mm_Vertical" H 3200 2000 50  0001 C CNN
+F 2 "Connector_PinSocket_2.54mm:PinSocket_1x19_P2.54mm_Vertical" H 3200 2000 50  0001 C CNN
 F 3 "~" H 3200 2000 50  0001 C CNN
 	1    3200 2000
@@
 F 0 "J4" H 1327 6076 50  0000 L CNN
 F 1 "EXT1_1" H 1327 5985 50  0000 L CNN
-F 2 "Connector_PinHeader_2.54mm:PinHeader_1x04_P2.54mm_Vertical" H 1300 6100 50  0001 C CNN
+F 2 "Connector_PinSocket_2.54mm:PinSocket_1x04_P2.54mm_Vertical" H 1300 6100 50  0001 C CNN
 F 3 "~" H 1300 6100 50  0001 C CNN
 	1    1300 6100
@@
 F 0 "J7" H 1327 6776 50  0000 L CNN
 F 1 "EXT2_1" H 1327 6685 50  0000 L CNN
-F 2 "Connector_PinHeader_2.54mm:PinHeader_1x06_P2.54mm_Vertical" H 1300 6800 50  0001 C CNN
+F 2 "Connector_PinSocket_2.54mm:PinSocket_1x06_P2.54mm_Vertical" H 1300 6800 50  0001 C CNN
 F 3 "~" H 1300 6800 50  0001 C CNN
 	1    1300 6800
@@
 F 0 "J5" H 2427 6076 50  0000 L CNN
 F 1 "EXT1_2" H 2427 5985 50  0000 L CNN
-F 2 "Connector_PinHeader_2.54mm:PinHeader_1x04_P2.54mm_Vertical" H 2400 6100 50  0001 C CNN
+F 2 "Connector_PinSocket_2.54mm:PinSocket_1x04_P2.54mm_Vertical" H 2400 6100 50  0001 C CNN
 F 3 "~" H 2400 6100 50  0001 C CNN
 	1    2400 6100
@@
 F 0 "J8" H 2427 6776 50  0000 L CNN
 F 1 "EXT2_2" H 2427 6685 50  0000 L CNN
-F 2 "Connector_PinHeader_2.54mm:PinHeader_1x06_P2.54mm_Vertical" H 2400 6800 50  0001 C CNN
+F 2 "Connector_PinSocket_2.54mm:PinSocket_1x06_P2.54mm_Vertical" H 2400 6800 50  0001 C CNN
 F 3 "~" H 2400 6800 50  0001 C CNN
 	1    2400 6800
@@
 F 0 "J6" H 3527 6076 50  0000 L CNN
 F 1 "EXT1_3" H 3527 5985 50  0000 L CNN
-F 2 "Connector_PinHeader_2.54mm:PinHeader_1x04_P2.54mm_Vertical" H 3500 6100 50  0001 C CNN
+F 2 "Connector_PinSocket_2.54mm:PinSocket_1x04_P2.54mm_Vertical" H 3500 6100 50  0001 C CNN
 F 3 "~" H 3500 6100 50  0001 C CNN
 	1    3500 6100
@@
 F 0 "J9" H 3527 6776 50  0000 L CNN
 F 1 "EXT2_3" H 3527 6685 50  0000 L CNN
-F 2 "Connector_PinHeader_2.54mm:PinHeader_1x06_P2.54mm_Vertical" H 3500 6800 50  0001 C CNN
+F 2 "Connector_PinSocket_2.54mm:PinSocket_1x06_P2.54mm_Vertical" H 3500 6800 50  0001 C CNN
 F 3 "~" H 3500 6800 50  0001 C CNN
 	1    3500 6800
@@
 	4600 6000 4600 5900
 Text Label 4500 5900 2    50   ~ 0
-GPIO13
+GPIO12
 Wire Wire Line
 	4500 5900 4600 5900
@@
 	4600 6500 4600 6400
 Text Label 4500 6400 2    50   ~ 0
-GPIO12
+GPIO13
 Wire Wire Line
 	4500 6400 4600 6400
@@
 	5700 6000 5700 5900
 Text Label 5600 5900 2    50   ~ 0
-GPIO15
+GPIO14
 Wire Wire Line
 	5600 5900 5700 5900
@@
 	5700 6500 5700 6400
 Text Label 5600 6400 2    50   ~ 0
-GPIO14
+GPIO15
 Wire Wire Line
 	5600 6400 5700 6400
@@
 	1    0    0    -1
 $EndComp
+$Comp
+L Mechanical:Housing N1
+U 1 1 5BE12A6D
+P 7700 6200
+F 0 "N1" H 7853 6234 50  0000 L CNN
+F 1 "Housing" H 7853 6143 50  0000 L CNN
+F 2 "custom_footprint:2.4INCH_TFT_LCD_18P_0.80mm_FOLD" H 7750 6250 50  0001 C CNN
+F 3 "~" H 7750 6250 50  0001 C CNN
+	1    7700 6200
+	1    0    0    -1
+$EndComp

Commit message: Arranged to v0.1
Parts:
- added D1: 0603/BLUE, LED_SMD:LED_0603_1608Metric, symbol Device:LED
- added D2: 0603/RED, LED_SMD:LED_0603_1608Metric, symbol Device:LED
- added H3, H4: MountingHole, MountingHole:MountingHole_8.4mm_M8, symbol Mechanical:MountingHole
- added R5: 0603/470R, Resistor_SMD:R_0603_1608Metric, symbol Device:R
- added R6: 0603/1K, Resistor_SMD:R_0603_1608Metric, symbol Device:R
- J4, J5, J6: footprint Connector_PinSocket_2.54mm:PinSocket_1x04_P2.54mm_Vertical -> custom_footprint:PinSocket_1x04_P2.54mm_Vertical_NO3D
- J7, J8, J9: footprint Connector_PinSocket_2.54mm:PinSocket_1x06_P2.54mm_Vertical -> custom_footprint:PinSocket_1x06_P2.54mm_Vertical_NO3D
- N1: value Housing -> 2.4\" LCD
- R4: value 0603/4.7 -> 0603/4.7R
Connections:
- net GND: now also R5.1, R6.1
- net GPIO32: now reaches J1.7 (Pin_7)
- net GPIO17: now reaches J2.11 (Pin_11)
- net GPIO17: now also D2.1 (K)
- net GPIO16: now reaches J2.12 (Pin_12)
- net GPIO16: now also D1.1 (K)
- new net: D1.2 (A), R5.2
- new net: D2.2 (A), R6.2
- no-connect marks 36 -> 54
Other:
- note added: "NOT FOR USE"
- moved on the sheet: H1, H2, J4, J5, J6, J7, J8, J9, N1
